Commit message: Lab 7 Task 4: Gazebo materials and diff drive plugin

File: Lab7/wojnae/webots_ws/install/my_robot/share/my_robot/urdf/my_robot.urdf.xacro (robot description, xacro)
@@ -129,5 +129,5 @@
       rpy="0 0 0"/>
   </link>
-  <joint name="base_left_wheel_joint" type="fixed">
+  <joint name="base_left_wheel_joint" type="continuous">
     <parent link="base_link"/>
     <child link="left_wheel"/>
@@ -155,5 +155,5 @@
       rpy="0 0 0"/>
   </link>
-  <joint name="base_right_wheel_joint" type="fixed">
+  <joint name="base_right_wheel_joint" type="continuous">
     <parent link="base_link"/>
     <child link="right_wheel"/>
@@ -185,3 +185,42 @@
     <origin xyz="0.25 0 -0.05" rpy="0 0 0"/>
   </joint>
+  <!-- ================= GAZEBO MATERIALS ================= -->
+  <gazebo reference="base_link">
+    <material>Gazebo/Green</material>
+  </gazebo>
+  <gazebo reference="left_wheel">
+    <material>Gazebo/Grey</material>
+  </gazebo>
+  <gazebo reference="right_wheel">
+    <material>Gazebo/Grey</material>
+  </gazebo>
+  <gazebo reference="caster_wheel">
+    <material>Gazebo/Grey</material>
+  </gazebo>
+  <gazebo reference="lidar">
+    <material>Gazebo/White</material>
+  </gazebo>
+  <!-- ================= DIFF DRIVE PLUGIN ================= -->
+  <gazebo>
+    <plugin name="diff_drive_controller"
+      filename="libgazebo_ros_diff_drive.so">
+      <!-- Update rate in Hz -->
+      <update_rate>50</update_rate>
+      <!-- Wheels -->
+      <left_joint>base_left_wheel_joint</left_joint>
+      <right_joint>base_right_wheel_joint</right_joint>
+      <!-- Kinematics -->
+      <wheel_separation>0.4</wheel_separation>
+      <wheel_diameter>0.2</wheel_diameter>
+      <!-- Output -->
+      <publish_odom>true</publish_odom>
+      <publish_odom_tf>true</publish_odom_tf>
+      <publish_wheel_tf>true</publish_wheel_tf>
+      <odometry_topic>odom</odometry_topic>
+      <odometry_frame>odom</odometry_frame>
+      <robot_base_frame>base_footprint</robot_base_frame>
+      <!-- Input -->
+      <command_topic>cmd_vel</command_topic>
+    </plugin>
+  </gazebo>
 </robot>
